File: kicad/hammerhead_turret_controller/coprocessor.kicad_sch (KiCad schematic)
At the start: 16 parts, among them IC1 STM32F302CBT6, J6 Conn_01x03, J8 SWD, Y1 ASDDV-24.000MHZ-LC-T

Commit message: add can transceiver
Connections:
- net CAN_FAULT: now reaches IC1.31 (PA10)
- net CAN_RX: now reaches IC1.32 (PA11)
- net CAN_TX: now reaches IC1.33 (PA12)
- net TC_I2C_SCL: no longer names the net of IC1.42 (PB6)
- net TC_I2C_SDA: no longer names the net of IC1.43 (PB7)
- no-connect marks 8 -> 7
Changed lines of the file:
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@@
-	)
-	(no_connect
-		(at 142.24 57.15)
 	)
 	(no_connect
@@
 	)
 	(no_connect
+		(at 142.24 85.09)
+	)
+	(no_connect
 		(at 185.42 76.2)
 	)
 	(no_connect
-		(at 142.24 54.61)
-	)
-	(no_connect
-		(at 142.24 59.69)
+		(at 142.24 82.55)
 	)
 	(wire
@@
 	(wire
 		(pts
-			(xy 128.27 82.55) (xy 142.24 82.55)
-		)
-		(stroke
-			(width 0)
-			(type default)
-		)
-	)
-	(wire
-		(pts
 			(xy 85.09 116.84) (xy 87.63 116.84)
 		)
@@
 	(wire
 		(pts
+			(xy 129.54 54.61) (xy 142.24 54.61)
+		)
+		(stroke
+			(width 0)
+			(type default)
+		)
+	)
+	(wire
+		(pts
+			(xy 129.54 57.15) (xy 142.24 57.15)
+		)
+		(stroke
+			(width 0)
+			(type default)
+		)
+	)
+	(wire
+		(pts
 			(xy 128.27 132.08) (xy 142.24 132.08)
 		)
@@
 	(wire
 		(pts
-			(xy 128.27 85.09) (xy 142.24 85.09)
+			(xy 129.54 59.69) (xy 142.24 59.69)
 		)
 		(stroke
@@
 		)
 	)
+	(label "CAN_TX"
+		(at 132.08 59.69 0)
+		(effects
+			(font
+				(size 1.27 1.27)
+			)
+			(justify left bottom)
+		)
+	)
 	(label "PAN_MS3"
 		(at 132.08 44.45 0)
@@
 		)
 	)
+	(label "CAN_FAULT"
+		(at 132.08 54.61 0)
+		(effects
+			(font
+				(size 1.27 1.27)
+			)
+			(justify left bottom)
+		)
+	)
 	(label "SPI_MISO"
 		(at 133.35 77.47 0)
@@
 		)
 	)
-	(label "TC_I2C_SCL"
-		(at 130.81 82.55 0)
-		(effects
-			(font
-				(size 1.27 1.27)
-			)
-			(justify left bottom)
-		)
-	)
 	(label "OSC_IN"
 		(at 134.62 116.84 0)
@@
 		)
 	)
+	(label "CAN_RX"
+		(at 132.08 57.15 0)
+		(effects
+			(font
+				(size 1.27 1.27)
+			)
+			(justify left bottom)
+		)
+	)
 	(label "SPI_MOSI"
 		(at 133.35 80.01 0)
@@
 	(label "FAULT_LED"
 		(at 132.08 97.79 0)
-		(effects
-			(font
-				(size 1.27 1.27)
-			)
-			(justify left bottom)
-		)
-	)
-	(label "TC_I2C_SDA"
-		(at 130.81 85.09 0)
 		(effects
 			(font
@@
 		)
 	)
-	(hierarchical_label "TC_I2C_SDA"
-		(shape bidirectional)
-		(at 128.27 85.09 180)
-		(effects
-			(font
-				(size 1.27 1.27)
-			)
-			(justify right)
-		)
-	)
 	(hierarchical_label "PAN_STEP"
 		(shape output)
@@
 		)
 	)
+	(hierarchical_label "CAN_FAULT"
+		(shape input)
+		(at 129.54 54.61 180)
+		(effects
+			(font
+				(size 1.27 1.27)
+			)
+			(justify right)
+		)
+	)
 	(hierarchical_label "GND"
 		(shape passive)
@@
 		)
 	)
-	(hierarchical_label "TC_I2C_SCL"
-		(shape bidirectional)
-		(at 128.27 82.55 180)
+	(hierarchical_label "CAN_TX"
+		(shape output)
+		(at 129.54 59.69 180)
 		(effects
 			(font
@@
 		(effects
 			(font
+				(size 1.27 1.27)
+			)
+			(justify right)
+		)
+	)
+	(hierarchical_label "CAN_RX"
+		(shape output)
+		(at 129.54 57.15 180)
+		(effects
+			(font
