File: kicad/hammerhead_turret_controller/hammerhead_turret_controller.kicad_pcb (KiCad board)
At the start: 4 copper layers, 88.5 x 21.5 mm, 101 parts, among them IC1 STM32F302CBT6, J1 PLATFORM_CONN, J2 B4B-XH-A, J3 B4B-XH-A, J4 B6B-XH-A_LF__SN_, J5 B6B-XH-A_LF__SN_, J6 Conn_01x03, J8 SWD, Q1 BSS138LT1G, Q2 BSS138LT1G, Q3 BSS138LT1G, Q4 BSS138LT1G, U1 MC3486DR, U10 A4988SETTR-T, U13 A4988SETTR-T, U7 RT9193-33GB, U8 BMI270, Y1 ASDDV-24.000MHZ-LC-T

Commit message: add can transceiver
Parts:
- removed C24: 1uF, Capacitor_SMD:C_0603_1608Metric
- removed C25: 22nF, Capacitor_SMD:C_0402_1005Metric
- removed C26: 0.1uF, Capacitor_SMD:C_0402_1005Metric
- removed C27: 10uF, Capacitor_SMD:C_0603_1608Metric
- removed C38: 0.1uF, Capacitor_SMD:C_0201_0603Metric
- removed C39, C40: 22uF, Capacitor_SMD:C_1206_3216Metric
- removed C41: 75pF, Capacitor_SMD:C_0201_0603Metric
- removed L2: NR6028T150M, NR6028T150M:NR6028T150M
- removed R28: 10k, Resistor_SMD:R_0402_1005Metric
- removed R33: 511k, Resistor_SMD:R_0201_0603Metric
- removed R34: 105k, Resistor_SMD:R_0201_0603Metric
- removed R35: 49.9k, Resistor_SMD:R_0201_0603Metric
- removed R36: 100k, Resistor_SMD:R_0201_0603Metric
- removed R37: 13.3k, Resistor_SMD:R_0201_0603Metric
- removed R41, R53: 22k, Resistor_SMD:R_0201_0603Metric
- removed R43, R55: 18k, Resistor_SMD:R_0201_0603Metric
- removed U7: RT9193-33GB, RT9193-33GB:SOT-23-5_RIT
- added C11: 0.1uF, Capacitor_SMD:C_0402_1005Metric, F.Cu at (179.9, 53.7)
- added C12: 22uF, Capacitor_SMD:C_1206_3216Metric, F.Cu at (185.4, 59.4)
- added C13: 10uF, Capacitor_SMD:C_0603_1608Metric, F.Cu at (179.3, 54.9)
- added C14: 75pF, Capacitor_SMD:C_0201_0603Metric, B.Cu at (189.7, 65.4)
- added C15: 0.1uF, Capacitor_SMD:C_0402_1005Metric, B.Cu at (188.3, 69.8)
- added C6: 1uF, Capacitor_SMD:C_0603_1608Metric, F.Cu at (179.3, 56.4)
- added C7: 0.1uF, Capacitor_SMD:C_0201_0603Metric, F.Cu at (188.9, 62.5)
- added C8: 22nF, Capacitor_SMD:C_0402_1005Metric, F.Cu at (185.2, 54.2)
- added C9: 22uF, Capacitor_SMD:C_1206_3216Metric, F.Cu at (187.7, 59.4)
- added L1: NR6028T150M, NR6028T150M:NR6028T150M, F.Cu at (180.2, 62.0)
- added R19: 22k, Resistor_SMD:R_0201_0603Metric, F.Cu at (201.2, 68.5)
- added R20: 10k, Resistor_SMD:R_0402_1005Metric, F.Cu at (185.2, 56.1)
- added R21: 49.9k, Resistor_SMD:R_0201_0603Metric, F.Cu at (189.7, 65.4)
- added R22: 100k, Resistor_SMD:R_0201_0603Metric, B.Cu at (188.9, 65.3)
- added R23: 13.3k, Resistor_SMD:R_0201_0603Metric, B.Cu at (187.9, 65.0)
- added R24: 10k, Resistor_SMD:R_0402_1005Metric, B.Cu at (189.2, 71.3)
- added R25: 120, Resistor_SMD:R_0603_1608Metric, F.Cu at (193.6, 69.8)
- added R26: 22k, Resistor_SMD:R_0201_0603Metric, F.Cu at (208.6, 68.5)
- added U2: RT9193-33GB, RT9193-33GB:SOT-23-5_RIT, F.Cu at (182.8, 55.1)
- added U3: TCAN337DR, TCAN337DR:D0008A_N, F.Cu at (189.2, 69.7)
- added VR3: 3314J-1-103E, 3314J-1-103E:TRIM_3314J-1-103E, F.Cu at (197.6, 69.7)
- added VR4: 3314J-1-103E, 3314J-1-103E:TRIM_3314J-1-103E, F.Cu at (204.9, 69.7)
- J1: value PLATFORM_CONN -> 430450812; footprint B4B-XH-A:JST_B4B-XH-A -> 430450812:CONN_SD-43045-005_08_MOL
- R1: value 2k -> 511k
- R2: value 2k -> 105k
- R5, R6, R7: moved to B.Cu
- moved R2 15.6 mm to (189.7, 63.9)
- moved R1 14.3 mm to (188.9, 63.9), turned to 90 degrees
- moved J1 4.44 mm to (172.5, 68.9), turned to 180 degrees
- moved R5 1.65 mm to (203.1, 65.9), turned to -90 degrees
- moved R7 1.00 mm to (206.2, 66.4)
- moved R6 1.00 mm to (199.9, 66.4)
- moved ? 0.70 mm to (135.6, 70.0)
- moved ? 0.70 mm to (218.6, 70.0)
Connections:
- IC1 pad 31: unconnected-(IC1-PA10-Pad31) -> /CAN_FAULT
- IC1 pad 32: unconnected-(IC1-PA11-Pad32) -> /CAN_RX
- IC1 pad 33: unconnected-(IC1-PA12-Pad33) -> /CAN_TX
- IC1 pad 42: /I2C_SCL -> unconnected-(IC1-PB6-Pad42)
- IC1 pad 43: /I2C_SDA -> unconnected-(IC1-PB7-Pad43)
- J1 pad 3: /I2C_SDA -> /CANH
- J1 pad 4: /I2C_SCL -> /CANL
- R1 pad 1: 3V3 -> Net-(PS1-EN)
- R1 pad 2: /I2C_SDA -> 14.8V
- R2 pad 1: 3V3 -> GND
- R2 pad 2: /I2C_SCL -> Net-(PS1-EN)
Routing:
- net Net-(U13-REF): track 2.08 -> 82.6 mm, vias 0 -> 2
- net Net-(U10-REF): track 1.92 -> 61.2 mm, vias 0 -> 2
- net /CAN_FAULT: track 0.00 -> 25.0 mm, vias 0 -> 4
- net /I2C_SDA: track 23.2 -> 0.00 mm, vias 2 -> 0
- net /CAN_RX: track 0.00 -> 22.6 mm, vias 0 -> 2
- net /I2C_SCL: track 21.9 -> 0.00 mm, vias 2 -> 0
- net 3V3: track 45.8 -> 66.1 mm, vias 30 -> 31
- net /CANH: track 0.00 -> 19.8 mm
- net /CAN_TX: track 0.00 -> 19.0 mm
- net /CANL: track 0.00 -> 16.1 mm
- net GND: track 35.1 -> 37.6 mm, vias 83 -> 86
- net Net-(C41-Pad1): track 2.37 -> 0.00 mm, vias 1 -> 0
- net Net-(C14-Pad1): track 0.00 -> 2.37 mm, vias 0 -> 1
- net Net-(R26-Pad2): track 0.00 -> 1.76 mm
- net Net-(U7-BP): track 1.49 -> 0.00 mm
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Other:
- board size 88.5 x 21.5 mm -> 88.5 x 25 mm
- board text added: "HTC Rev B"
- board text removed: "HTC Rev A"
