File: kicad/hammerhead_turret_controller/power.kicad_sch (KiCad schematic)
At the start: 19 parts, among them U7 RT9193-33GB

Commit message: add can transceiver
Parts:
- renumbered C26 to C11, C40 to C12, C27 to C13, C41 to C14, C24 to C6, C38 to C7, C25 to C8, C39 to C9, L2 to L1, R33 to R1, R34 to R2, R28 to R20, R35 to R21, R36 to R22, R37 to R23, U7 to U2
Changed lines of the file:
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@@
 		(dnp no)
 		(fields_autoplaced yes)
-		(property "Reference" "C38"
+		(property "Reference" "C7"
 			(at 134.62 46.99 90)
 			(effects
@@
 		)
 		(instances
-			(project ""
-				(path "/28590d3f-7223-4dd1-9b76-1216899ace6a/c56623c0-cbed-4c5d-8242-113102137fec"
-					(reference "C38")
+			(project "hammerhead_turret_controller"
+				(path "/28590d3f-7223-4dd1-9b76-1216899ace6a/c56623c0-cbed-4c5d-8242-113102137fec"
+					(reference "C7")
 					(unit 1)
 				)
@@
 		(dnp no)
 		(fields_autoplaced yes)
-		(property "Reference" "R36"
+		(property "Reference" "R22"
 			(at 199.39 74.9299 0)
 			(effects
@@
 			(project "hammerhead_turret_controller"
 				(path "/28590d3f-7223-4dd1-9b76-1216899ace6a/c56623c0-cbed-4c5d-8242-113102137fec"
-					(reference "R36")
+					(reference "R22")
 					(unit 1)
 				)
@@
 		(on_board yes)
 		(dnp no)
-		(property "Reference" "C25"
+		(property "Reference" "C8"
 			(at 147.574 140.97 0)
 			(effects
@@
 			(project "hammerhead_turret_controller"
 				(path "/28590d3f-7223-4dd1-9b76-1216899ace6a/c56623c0-cbed-4c5d-8242-113102137fec"
-					(reference "C25")
+					(reference "C8")
 					(unit 1)
 				)
@@
 		(on_board yes)
 		(dnp no)
-		(property "Reference" "R28"
+		(property "Reference" "R20"
 			(at 131.826 142.24 0)
 			(effects
@@
 			(project "hammerhead_turret_controller"
 				(path "/28590d3f-7223-4dd1-9b76-1216899ace6a/c56623c0-cbed-4c5d-8242-113102137fec"
-					(reference "R28")
+					(reference "R20")
 					(unit 1)
 				)
@@
 		(on_board yes)
 		(dnp no)
-		(property "Reference" "C27"
+		(property "Reference" "C13"
 			(at 185.674 135.636 0)
 			(effects
@@
 			(project "hammerhead_turret_controller"
 				(path "/28590d3f-7223-4dd1-9b76-1216899ace6a/c56623c0-cbed-4c5d-8242-113102137fec"
-					(reference "C27")
+					(reference "C13")
 					(unit 1)
 				)
@@
 		(on_board yes)
 		(dnp no)
-		(property "Reference" "C24"
+		(property "Reference" "C6"
 			(at 83.312 136.144 0)
 			(effects
@@
 			(project "hammerhead_turret_controller"
 				(path "/28590d3f-7223-4dd1-9b76-1216899ace6a/c56623c0-cbed-4c5d-8242-113102137fec"
-					(reference "C24")
+					(reference "C6")
 					(unit 1)
 				)
@@
 		(dnp no)
 		(fields_autoplaced yes)
-		(property "Reference" "R37"
+		(property "Reference" "R23"
 			(at 199.39 86.3599 0)
 			(effects
@@
 			(project "hammerhead_turret_controller"
 				(path "/28590d3f-7223-4dd1-9b76-1216899ace6a/c56623c0-cbed-4c5d-8242-113102137fec"
-					(reference "R37")
+					(reference "R23")
 					(unit 1)
 				)
@@
 		(dnp no)
 		(fields_autoplaced yes)
-		(property "Reference" "R35"
+		(property "Reference" "R21"
 			(at 199.39 64.7699 0)
 			(effects
@@
 		)
 		(instances
-			(project ""
-				(path "/28590d3f-7223-4dd1-9b76-1216899ace6a/c56623c0-cbed-4c5d-8242-113102137fec"
-					(reference "R35")
+			(project "hammerhead_turret_controller"
+				(path "/28590d3f-7223-4dd1-9b76-1216899ace6a/c56623c0-cbed-4c5d-8242-113102137fec"
+					(reference "R21")
 					(unit 1)
 				)
@@
 		(dnp no)
 		(fields_autoplaced yes)
-		(property "Reference" "C40"
+		(property "Reference" "C12"
 			(at 180.34 64.7699 0)
 			(effects
@@
 		)
 		(instances
-			(project ""
-				(path "/28590d3f-7223-4dd1-9b76-1216899ace6a/c56623c0-cbed-4c5d-8242-113102137fec"
-					(reference "C40")
+			(project "hammerhead_turret_controller"
+				(path "/28590d3f-7223-4dd1-9b76-1216899ace6a/c56623c0-cbed-4c5d-8242-113102137fec"
+					(reference "C12")
 					(unit 1)
 				)
@@
 		(on_board yes)
 		(dnp no)
-		(property "Reference" "C39"
+		(property "Reference" "C9"
 			(at 167.64 64.7699 0)
 			(effects
@@
 		)
 		(instances
-			(project ""
-				(path "/28590d3f-7223-4dd1-9b76-1216899ace6a/c56623c0-cbed-4c5d-8242-113102137fec"
-					(reference "C39")
+			(project "hammerhead_turret_controller"
+				(path "/28590d3f-7223-4dd1-9b76-1216899ace6a/c56623c0-cbed-4c5d-8242-113102137fec"
+					(reference "C9")
 					(unit 1)
 				)
@@
 		(dnp no)
 		(fields_autoplaced yes)
-		(property "Reference" "R34"
+		(property "Reference" "R2"
 			(at 90.17 74.9299 0)
 			(effects
@@
 		)
 		(instances
-			(project ""
-				(path "/28590d3f-7223-4dd1-9b76-1216899ace6a/c56623c0-cbed-4c5d-8242-113102137fec"
-					(reference "R34")
+			(project "hammerhead_turret_controller"
+				(path "/28590d3f-7223-4dd1-9b76-1216899ace6a/c56623c0-cbed-4c5d-8242-113102137fec"
+					(reference "R2")
 					(unit 1)
 				)
@@
 		)
 		(instances
-			(project ""
+			(project "hammerhead_turret_controller"
 				(path "/28590d3f-7223-4dd1-9b76-1216899ace6a/c56623c0-cbed-4c5d-8242-113102137fec"
 					(reference "C1")
@@
 		(dnp no)
 		(fields_autoplaced yes)
-		(property "Reference" "R33"
+		(property "Reference" "R1"
 			(at 90.17 57.1499 0)
 			(effects
@@
 		)
 		(instances
-			(project ""
-				(path "/28590d3f-7223-4dd1-9b76-1216899ace6a/c56623c0-cbed-4c5d-8242-113102137fec"
-					(reference "R33")
+			(project "hammerhead_turret_controller"
+				(path "/28590d3f-7223-4dd1-9b76-1216899ace6a/c56623c0-cbed-4c5d-8242-113102137fec"
+					(reference "R1")
 					(unit 1)
 				)
@@
 		(dnp no)
 		(fields_autoplaced yes)
-		(property "Reference" "C41"
+		(property "Reference" "C14"
 			(at 213.36 74.9299 0)
 			(effects
@@
 		)
 		(instances
-			(project ""
-				(path "/28590d3f-7223-4dd1-9b76-1216899ace6a/c56623c0-cbed-4c5d-8242-113102137fec"
-					(reference "C41")
+			(project "hammerhead_turret_controller"
+				(path "/28590d3f-7223-4dd1-9b76-1216899ace6a/c56623c0-cbed-4c5d-8242-113102137fec"
+					(reference "C14")
 					(unit 1)
 				)
@@
 		(on_board yes)
 		(dnp no)
-		(property "Reference" "C26"
+		(property "Reference" "C11"
 			(at 166.116 135.636 0)
 			(effects
@@
 			(project "hammerhead_turret_controller"
 				(path "/28590d3f-7223-4dd1-9b76-1216899ace6a/c56623c0-cbed-4c5d-8242-113102137fec"
-					(reference "C26")
+					(reference "C11")
 					(unit 1)
 				)
@@
 		(dnp no)
 		(fields_autoplaced yes)
-		(property "Reference" "U7"
+		(property "Reference" "U2"
 			(at 118.11 120.65 0)
 			(effects
@@
 			(project "hammerhead_turret_controller"
 				(path "/28590d3f-7223-4dd1-9b76-1216899ace6a/c56623c0-cbed-4c5d-8242-113102137fec"
-					(reference "U7")
+					(reference "U2")
 					(unit 1)
 				)
@@
 		)
 		(instances
-			(project ""
+			(project "hammerhead_turret_controller"
 				(path "/28590d3f-7223-4dd1-9b76-1216899ace6a/c56623c0-cbed-4c5d-8242-113102137fec"
 					(reference "PS1")
@@
 		(dnp no)
 		(fields_autoplaced yes)
-		(property "Reference" "L2"
+		(property "Reference" "L1"
 			(at 150.114 55.626 0)
 			(effects
@@
 		)
 		(instances
-			(project ""
-				(path "/28590d3f-7223-4dd1-9b76-1216899ace6a/c56623c0-cbed-4c5d-8242-113102137fec"
-					(reference "L2")
+			(project "hammerhead_turret_controller"
+				(path "/28590d3f-7223-4dd1-9b76-1216899ace6a/c56623c0-cbed-4c5d-8242-113102137fec"
+					(reference "L1")
 					(unit 1)
 				)
@@
 		)
 		(instances
-			(project ""
+			(project "hammerhead_turret_controller"
 				(path "/28590d3f-7223-4dd1-9b76-1216899ace6a/c56623c0-cbed-4c5d-8242-113102137fec"
 					(reference "C2")
